File: picdiv_board_v3.kicad_sch (KiCad schematic)
At the start: 81 parts, among them J1 DC-Input, J10 PPS_B, J14 TEST_1PPS, J4 SYNC, J6 PPS_B, J8 SYNC, Q1 Q_PNP_BEC, Q2 Q_PNP_BEC, U1 LT1963AxST-3.3, U2 LT1963AxST-3.3, U3 PIC12F675, U6 IDT5PB1108

Commit message: kicad7
Parts:
- gave numbers to parts that had none: 27
